Commit message: Add files via upload
the new pkg after mapping (shehab's version)

File: WAFL2025/urdf/WAFL2025.urdf (robot description, URDF)
Before this commit: robot WAFL2025, 11 links, 10 joints
Links:
- removed link base_footprint
- removed link hokuyo_link
- added link rplidar_link, mass 0.5; collision cylinder length=0.07 radius=0.05; visual cylinder length=0.07 radius=0.05
Joints:
- removed joint chassis_base_footprint
- removed joint hokuyo_joint
- added joint rplidar_joint: type fixed, parent base_link, child rplidar_link, origin xyz=0.59 0 0.5 rpy=0 0 0

Commit message: Add files via upload
Last Version with AMCL and added path planning

File: WAFL2025/urdf/WAFL2025.urdf (robot description, URDF)
Before this commit: robot WAFL2025, 10 links, 9 joints
Links:
- link rplidar_link: geometry collision cylinder length=0.06 radius=0.05; visual cylinder length=0.06 radius=0.05

Commit message: Add files via upload
last version of autonomous module of team WAFL25

File: WAFL2025/urdf/WAFL2025.urdf (robot description, URDF)
Before this commit: robot WAFL2025, 11 links, 10 joints
Links:
- removed link base_footprint
- removed link hokuyo_link
- added link rplidar_link, mass 0.5; collision cylinder length=0.06 radius=0.05; visual cylinder length=0.06 radius=0.05
Joints:
- removed joint chassis_base_footprint
- removed joint hokuyo_joint
- added joint rplidar_joint: type fixed, parent base_link, child rplidar_link, origin xyz=0.59 0 0.5 rpy=0 0 0
